Commit message: Added urdf

File: src/robotics_toolbox/robots/robot_hw.urdf (robot description, URDF)
Before this commit: robot simple_robot, 2 links, 1 joints
Links:
- removed link end_effector
- added link cylinder_1; visual cylinder length=0.5 radius=0.05
- added link cylinder_2; visual cylinder length=0.250 radius=0.05
- added link cylinder_3; visual cylinder length=0.250 radius=0.05
- added link cylinder_4; visual cylinder length=0.250 radius=0.05
- added link ee
- added link sphere_1; visual sphere radius=0.06
- added link sphere_2; visual sphere radius=0.06
- link base_link: geometry visual box size=0.3 0.3 0.3
Joints:
- removed joint joint0
- added joint fixed_2: type fixed, parent cylinder_1, child sphere_1, origin xyz=0 0 0.5 rpy=0 0 0
- added joint fixed_3: type fixed, parent cylinder_3, child sphere_2, origin xyz=0 0 0.25 rpy=0 0 0
- added joint fixed_5: type fixed, parent cylinder_4, child ee, origin xyz=0 0 0.25 rpy=0 0 0
- added joint revolute_1: type revolute, parent base_link, child cylinder_1, origin xyz=0 0 0.15 rpy=0 0 0, axis 0 0 1, limit lower=-1.57 upper=1.57 effort=30 velocity=1.0
- added joint revolute_2: type revolute, parent sphere_1, child cylinder_2, origin xyz=0 0 0.0 rpy=0 0 0, axis 1 0 0, limit lower=-1.57 upper=1.57 effort=30 velocity=1.0
- added joint revolute_3: type revolute, parent cylinder_2, child cylinder_3, origin xyz=0 0 0.25 rpy=0 0 0, axis 0 0 1, limit lower=-1.57 upper=1.57 effort=30 velocity=1.0
- added joint revolute_4: type revolute, parent sphere_2, child cylinder_4, origin xyz=0 0 0.0 rpy=0 0 0, axis 1 0 0, limit lower=-1.57 upper=1.57 effort=30 velocity=1.0
